File: hardware/GuardianSense.kicad_pcb (KiCad board)
At the start: 2 copper layers, 54 x 85 mm, 23 parts, among them P1 USB_C_Plug_USB2.0, SW1 SW_SPST, SW2 SW_SPST, U1 ESP32-S3-WROOM-1, U2 D3V3XA4B10LP, U3 AMS1117-3.3

Commit message: Sunday Fun!
Parts:
- added C7: 0.1uF, Capacitor_SMD:C_0805_2012Metric, F.Cu at (143.1, 112.1)
- added C8: 0.1uF, Capacitor_SMD:C_0805_2012Metric, F.Cu at (143.1, 115.1)
- added JP1: SolderJumper_2_Open, Jumper:SolderJumper-2_P1.3mm_Open_TrianglePad1.0x1.5mm, F.Cu at (143.0, 118.4)
- added R5: 4.7k, Resistor_SMD:R_0805_2012Metric, F.Cu at (147.5, 112.1)
- added R6: 4.7k, Resistor_SMD:R_0805_2012Metric, F.Cu at (147.5, 115.0)
- added U4: BME280, Package_LGA:Bosch_LGA-8_2.5x2.5mm_P0.65mm_ClockwisePinNumbering, F.Cu at (147.6, 118.8)
- P1: footprint Connector_USB:USB_C_Receptacle_HRO_TYPE-C-31-M-12 -> Connector:USB-SMD_USB-TYPE-C-020
- moved C2 14.4 mm to (138.2, 106.4)
- moved C5 14.4 mm to (138.2, 115.4)
- moved C1 14.4 mm to (138.2, 103.4)
- moved C3 14.4 mm to (138.2, 109.4)
- moved C4 14.4 mm to (138.2, 112.4)
- moved C6 14.4 mm to (138.2, 118.4)
- moved D1 14.4 mm to (137.8, 86.9)
- moved R3 14.4 mm to (141.3, 86.9)
- moved U3 14.4 mm to (140.6, 94.9)
- moved P1 9.42 mm to (139.3, 74.2)
- moved U2 7.81 mm to (147.3, 73.8)
Connections:
- U1 pad 1: Net-(U1-GND-Pad1) -> GND
- U1 pad 13: /D_M -> /USB_M
- U1 pad 14: /D_P -> /USB_P
- U1 pad 40: Net-(U1-GND-Pad1) -> GND
- U1 pad 41: Net-(U1-GND-Pad1) -> GND
- U1 pad 8: /GPIO15 -> /I2C_SCL
- U1 pad 9: /GPIO16 -> /I2C_SDA
- U2 pad 10: unconnected-(U2-NC-Pad10) -> /USB_M
- U2 pad 7: unconnected-(U2-NC-Pad7) -> /USB_5V
- U2 pad 9: unconnected-(U2-NC-Pad9) -> /USB_P
Routing:
- net /USB_M: track 0.00 -> 13.7 mm
- net /USB_P: track 0.00 -> 5.29 mm
- added copper zone on B.Cu, net GND

Commit message: Updates Monday
Parts:
- added C10: 0.1uF, Capacitor_SMD:C_0805_2012Metric, F.Cu at (222.1, 62.9)
- added C11: 0.1uF, Capacitor_SMD:C_0805_2012Metric, F.Cu at (222.1, 66.0)
- added C8: 0.1uF, Capacitor_SMD:C_0805_2012Metric, F.Cu at (260.9, 111.9)
- added C9: 0.1uF, Capacitor_SMD:C_0805_2012Metric, F.Cu at (222.1, 59.9)
- added D4: SS14, Diode_SMD:D_SMA, F.Cu at (211.5, 74.2)
- added J1: Conn_01x03_Pin AM312 Module, Connector_PinHeader_2.54mm:PinHeader_1x03_P2.54mm_Vertical, F.Cu at (261.0, 103.0)
- added J2: Micro_SD_Card, Library:AMPHENOL_GTFP08431BEU, F.Cu at (171.4, 126.0)
- added LS1: MLT-8530, Library:MLT8530, F.Cu at (213.6, 65.6)
- added Q1: BC847, Package_TO_SOT_SMD:SOT-23, F.Cu at (222.3, 69.9)
- added R10: 10K, Resistor_SMD:R_0805_2012Metric, F.Cu at (256.5, 117.0)
- added R11: 10K, Resistor_SMD:R_0805_2012Metric, F.Cu at (256.5, 119.9)
- added R5: 1K, Resistor_SMD:R_0805_2012Metric, F.Cu at (256.5, 102.2)
- added R6: 1K, Resistor_SMD:R_0805_2012Metric, F.Cu at (256.5, 105.2)
- added R7: 10k, Resistor_SMD:R_0805_2012Metric, F.Cu at (256.5, 108.1)
- added R8: 10k, Resistor_SMD:R_0805_2012Metric, F.Cu at (256.5, 111.0)
- added R9: 10K, Resistor_SMD:R_0805_2012Metric, F.Cu at (256.5, 114.0)
- C1, C2: footprint Capacitor_SMD:C_0805_2012Metric -> Capacitor_SMD:CP_Elec_4x5.4
- moved C2 32.8 mm to (169.5, 96.7), turned to -90 degrees
- moved U3 20.6 mm to (161.2, 96.5)
- moved C1 16.7 mm to (153.5, 96.7), turned to -90 degrees
- moved R4 12.8 mm to (143.1, 108.5)
Connections:
- U4 pad 5: Net-(JP1-A) -> GND
Routing:
- removed copper zone on B.Cu, net GND

Commit message: Updates
Parts:
- removed the C8 at (143.1, 115.1)
- removed the C8 at (260.9, 111.9)
- removed J2: Micro_SD_Card, Library:AMPHENOL_GTFP08431BEU
- removed JP1: SolderJumper_2_Open, Jumper:SolderJumper-2_P1.3mm_Open_TrianglePad1.0x1.5mm
- removed LS1: MLT-8530, Library:MLT8530
- removed P1: USB_C_Plug_USB2.0, Connector:USB-SMD_USB-TYPE-C-020
- removed the R5 at (147.5, 112.1)
- removed the R5 at (256.5, 102.2)
- removed the R6 at (147.5, 115.0)
- removed the R6 at (256.5, 105.2)
- added C8: 0.1uF, Capacitor_SMD:C_0805_2012Metric, F.Cu at (83.8, 74.3)
- added R5: 1K, Resistor_SMD:R_0805_2012Metric, F.Cu at (70.6, 80.0)
- added R6: 1K, Resistor_SMD:R_0805_2012Metric, F.Cu at (70.6, 83.0)
- moved R10 185.9 mm to (75.0, 77.1)
- moved R11 185.9 mm to (75.0, 80.0)
- moved R7 185.9 mm to (75.0, 68.2)
- moved R8 185.9 mm to (75.0, 71.2)
- moved R9 185.9 mm to (75.0, 74.1)
- moved J1 147.7 mm to (117.3, 69.1)
- moved C10 134.1 mm to (88.3, 71.3)
- moved C11 134.1 mm to (88.3, 74.3)
- moved C9 134.1 mm to (88.3, 68.3)
- moved H4 101.8 mm to (121.0, 49.5)
- moved Q1 100.3 mm to (122.0, 69.2)
- moved D4 92.6 mm to (119.0, 78.7)
- moved H3 89.0 mm to (121.0, 42.4)
- moved U3 80.8 mm to (82.1, 80.0), turned to 0 degrees
- moved D2 79.3 mm to (103.1, 70.1), turned to 0 degrees
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Routing:
- net /USB_M: track 13.7 -> 0.00 mm
- net /USB_P: track 5.29 -> 0.00 mm
- net Net-(D1-A): track 1.62 -> 0.00 mm
