File: hardware/GuardianSense.kicad_sch (KiCad schematic)
At the start: 23 parts, among them P1 USB_C_Plug_USB2.0, SW1 SW_SPST, SW2 SW_SPST, U1 ESP32-S3-WROOM-1, U2 D3V3XA4B10LP, U3 AMS1117-3.3

Commit message: Sunday Fun!
Parts:
- added C7, C8: 0.1uF, Capacitor_SMD:C_0805_2012Metric, symbol Device:C
- added JP1: SolderJumper_2_Open, Jumper:SolderJumper-2_P1.3mm_Open_TrianglePad1.0x1.5mm, symbol Jumper:SolderJumper_2_Open
- added R5, R6: 4.7k, Resistor_SMD:R_0805_2012Metric, symbol Device:R
- added R7, R8: 10k, symbol Device:R
- added R9: R, symbol Device:R
- added U4: BME280, Package_LGA:Bosch_LGA-8_2.5x2.5mm_P0.65mm_ClockwisePinNumbering, symbol Sensor:BME280
- P1: footprint Connector_USB:USB_C_Receptacle_HRO_TYPE-C-31-M-12 -> Connector:USB-SMD_USB-TYPE-C-020
Connections:
- net D_M is gone; now on net USB_M: U1.13 (USB_D-)
- net D_P is gone; now on net USB_P: U1.14 (USB_D+)
- net GND: now also U1.1 (GND), U1.40 (GND), U1.41 (GND), C7.2, C8.2, R9.2, U4.1 (GND), U4.7 (GND)
- net USB_5V: now also U2.7 (NC)
- net USB_M: now also U2.10 (NC)
- net USB_P: now also U2.9 (NC)
- net VCC_3V3: now also C7.1, C8.1, JP1.2 (B), R5.2, R6.1, R7.1, R8.1, U4.2 (CSB), U4.6 (VDDIO), U4.8 (VDD)
- net GPIO15 renamed I2C_SCL
- net I2C_SCL: now also R6.2, R8.2, U4.4 (SCK)
- net GPIO16 renamed I2C_SDA
- net I2C_SDA: now also R5.1, R7.2, U4.3 (SDI)
- new net: JP1.1 (A), R9.1, U4.5 (SDO)

Commit message: Updates Monday
Parts:
- removed JP1: SolderJumper_2_Open, Jumper:SolderJumper-2_P1.3mm_Open_TrianglePad1.0x1.5mm, symbol Jumper:SolderJumper_2_Open
- added C10, C11, C9: 0.1uF, Capacitor_SMD:C_0805_2012Metric, symbol Device:C
- added D4: SS14, Diode_SMD:D_SMA, symbol Diode:SS14
- added J1: Conn_01x03_Pin AM312 Module, Connector_PinHeader_2.54mm:PinHeader_1x03_P2.54mm_Vertical, symbol Connector:Conn_01x03_Pin
- added J2: Micro_SD_Card, Library:AMPHENOL_GTFP08431BEU, symbol Connector:Micro_SD_Card
- added LS1: MLT-8530, Library:MLT8530, symbol FelipeLib:MLT-8530
- added Q1: BC847, Package_TO_SOT_SMD:SOT-23, symbol Transistor_BJT:BC847
- added R10, R11: 10K, Resistor_SMD:R_0805_2012Metric, symbol Device:R
- C1, C2: footprint Capacitor_SMD:C_0805_2012Metric -> Capacitor_SMD:CP_Elec_4x5.4
- R5, R6: value 4.7k -> 1K
- R7, R8: footprint (none) -> Resistor_SMD:R_0805_2012Metric
- R9: value R -> 10K; footprint (none) -> Resistor_SMD:R_0805_2012Metric
Connections:
- net GND: now also U4.5 (SDO), C10.2, C11.2, C9.2, J1.3 (Pin_3), J2.6 (VSS), J2.9 (SHIELD), Q1.2 (E); no longer C8.2, R9.2
- net GPIO14: now also R9.2, J2.5 (CLK)
- net GPIO2: now also J2.7 (DAT0), R11.2
- net GPIO38: now also J1.2 (Pin_2)
- net GPIO41: now also R5.1
- net I2C_SCL: no longer R6.2
- net I2C_SDA: no longer R5.1
- net USB_5V: now also R6.2, C9.1, D4.1 (K), J1.1 (Pin_1), LS1.2 (+LEAD)
- net VCC_3V3: now also C8.2, C10.1, C11.1; no longer C8.1, R5.2, R6.1
- net at R9.1: now also C8.1, J2.1 (DAT2), J2.2 (DAT3/CD), J2.4 (VDD), J2.8 (DAT1), R10.1, R11.1; no longer U4.5 (SDO)
- new net: D4.2 (A), LS1.3 (-LEAD), Q1.3 (C), R6.1
- new net: Q1.1 (B), R5.2
- new net GPIO15: J2.3 (CMD), R10.2
- no-connect marks 2 -> 4
Other:
- moved on the sheet: C2, C7, D1, R3

Commit message: Updates
Parts:
- P1: symbol Connector:USB_C_Plug_USB2.0 -> Connector:USB_C_Receptacle
Connections:
- net USB_M: now also P1.B7 (D-)
- net USB_P: now also P1.B6 (D+)
Other:
- moved on the sheet: R1, R2
